File: sboxnet-weichenservo/v1-sboxnet-weichenservo.sch (KiCad schematic (older format))
At the start: 34 parts, among them J1 Screw_Terminal_01x02, J10 Conn_01x03_Male, J11 Conn_01x03_Male, J12 Conn_01x03_Male, J13 Conn_02x08_Top_Bottom, J2 Screw_Terminal_01x04, J3 Conn_02x17_Odd_Even, J4 Screw_Terminal_01x04, J5 Conn_01x03_Male, J6 Conn_01x03_Male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

Commit message: v2-sboxnet-weichenservo
Parts:
- removed U1: L7805 CV 1.5A, symbol Regulator_Linear:L7805
- added U1: uA7805 D2PAK, Package_TO_SOT_SMD:ATPAK-2, symbol Regulator_Linear:uA7805
- D3: footprint Diode_SMD:D_SOD-323_HandSoldering -> Diode_SMD:D_SOD-323F
Changed lines of the file:
@@
 F 0 "D3" H 6650 1833 50  0000 C CNN
 F 1 "BAT 54J NXP" H 6550 1915 50  0000 C CNN
-F 2 "Diode_SMD:D_SOD-323_HandSoldering" H 6650 2050 50  0001 C CNN
+F 2 "Diode_SMD:D_SOD-323F" H 6650 2050 50  0001 C CNN
 F 3 "~" H 6650 2050 50  0001 C CNN
 	1    6650 2050
@@
 	6200 2050 6500 2050
 Connection ~ 6500 2050
+$Comp
+L Regulator_Linear:uA7805 U1
+U 1 1 60BBDD07
+P 2950 3050
+F 0 "U1" H 2950 3292 50  0000 C CNN
+F 1 "uA7805 D2PAK" H 2950 3201 50  0000 C CNN
+F 2 "Package_TO_SOT_SMD:ATPAK-2" H 2975 2900 50  0001 L CIN
+F 3 "http://www.ti.com/lit/ds/symlink/ua78.pdf" H 2950 3000 50  0001 C CNN
+	1    2950 3050
+	1    0    0    -1
+$EndComp
 Wire Wire Line
 	2200 3050 2650 3050
@@
 Wire Bus Line
 	2800 6600 2800 7700
-$Comp
-L Regulator_Linear:L7805 U1
-U 1 1 6141E933
-P 2950 3050
-F 0 "U1" H 2950 3292 50  0000 C CNN
-F 1 "L7805 CV 1.5A" H 2950 3201 50  0000 C CNN
-F 2 "" H 2975 2900 50  0001 L CIN
-F 3 "http://www.st.com/content/ccc/resource/technical/document/datasheet/41/4f/b3/b0/12/d4/47/88/CD00000444.pdf/files/CD00000444.pdf/jcr:content/translations/en.CD00000444.pdf" H 2950 3000 50  0001 C CNN
-	1    2950 3050
-	1    0    0    -1
-$EndComp
 $EndSCHEMATC
