File: sboxnet-dccgen/sboxnet-dccgen.sch (KiCad schematic (older format))
At the start: 15 parts, among them J1 sboxnet-stecker_02x17, J2 Screw_Terminal_01x02, U1 SN65HVD230

Commit message: neuer DCCGEN mit sboxnet Verteiler und Abschlusswiderstanden
Parts:
- added J10, J4, J5, J6, J8: 8P8C, sboxnet:8p8c-mebp, symbol Connector:8P8C
- added J11, J12, J3, J7, J9: Conn_01x02, Connector_PinHeader_2.54mm:PinHeader_1x02_P2.54mm_Vertical, symbol Connector_Generic:Conn_01x02
- added R10, R8, R9: 120, Resistor_SMD:R_1206_3216Metric, symbol Device:R
- D1: value LED -> gn
- D2: value LED -> rt
- R3: value 2,2k -> 1k
- R4, R5: value 680 -> 470
Connections:
- net +3V3: no longer R6.2, R7.2
- net DCC_A: now also R8.2; no longer R6.1
- net DCC_B: now also J3.2 (Pin_2); no longer R7.1
- new net: J3.1 (Pin_1), R8.1
- new net: J10.4, J12.2 (Pin_2)
- new net: J10.5, R10.1
- new net: J10.7, J11.2 (Pin_2)
- new net: J10.8, R9.1
- new net: J11.1 (Pin_1), R9.2
- new net: J12.1 (Pin_1), R10.2
- new net: J7.1 (Pin_1), R6.1
- new net: J9.1 (Pin_1), R7.1
- new net +7_x: J4.2, J4.3, J5.2, J5.3, J6.2, J6.3, J8.2, J8.3
- new net can_h_x: J4.5, J5.5, J6.5, J7.2 (Pin_2), J8.5
- new net can_l_x: J4.4, J5.4, J6.4, J8.4, R6.2
- new net dcc_a_x: J4.7, J5.7, J6.7, J8.7, R7.2
- new net dcc_b_x: J4.8, J5.8, J6.8, J8.8, J9.2 (Pin_2)
- new net gnd_x: J4.1, J4.6, J5.1, J5.6, J6.1, J6.6, J8.1, J8.6
Other:
- note removed: "gn"
- note removed: "rt"
- moved on the sheet: TP2, TP3
