File: sboxnet-booster/sboxnet-booster.sch (KiCad schematic (older format))
At the start: 67 parts, among them J1 sboxnet-stecker_02x17, J3 Conn_01x02_Male, J4 Conn_01x02_Male, J5 Screw_Terminal_01x04, J6 Screw_Terminal_01x04, J7 Power von externen 15V/4A Net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, SW1 Öffner, U1 L6206PSO-sboxnet, U2 L78L12_SOT89, U3 SN65HVD230

Commit message: booster modul mit l6206 dip
Parts:
- removed J1: sboxnet-stecker_02x17, sboxnet:sboxnet-stecker-2x17, symbol sboxnet:sboxnet-stecker_02x17
- added C11: 220n, Capacitor_SMD:C_1206_3216Metric, symbol Device:C
- added C12: 10n, Capacitor_SMD:C_1206_3216Metric, symbol Device:C
- added D14, D15: 1N4148WS, Diode_SMD:D_SOD-323, symbol Diode:1N4148WS
- added J?: sboxnet-stecker_02x17, symbol sboxnet:sboxnet-stecker_02x17
- added JP? (x3): SolderJumper_3_Open, symbol Jumper:SolderJumper_3_Open
- added R24: 100, Resistor_SMD:R_1206_3216Metric, symbol Device:R
- added R25, R27: 0.22, Resistor_THT:R_Axial_Power_L38.0mm_W9.0mm_P45.72mm, symbol Device:R
- added R26, R28: 10k, Resistor_THT:R_Axial_Power_L38.0mm_W9.0mm_P45.72mm, symbol Device:R
- added U4: l6206, symbol sboxnet:l6206
Connections:
- net labels added: Abschaltung_LED, DCC_IN, NOTAUS, NOTAUS_LED, OVERCUR, Overflow_LED, PB0, PB1, PB2
- net labels removed: +5V
- wire segments 152 -> 169
- no-connect marks 18 -> 16
Other:
- note added: "PB2..0 ModulCodierung\n"
- note added: "gn"
