File: sboxnet-booster/sboxnet-booster.kicad_pcb (KiCad board)
At the start: 2 copper layers, 114.3 x 110.5 mm, 67 parts, among them J1 sboxnet-stecker_02x17, J3 Conn_01x02_Male, J4 Conn_01x02_Male, J5 Screw_Terminal_01x04, J6 Screw_Terminal_01x04, J7 Power von externen 15V/4A Net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, SW1 Öffner, U1 L6206PSO-sboxnet, U2 L78L12_SOT89, U3 SN65HVD230

Commit message: IN1 and IN2 fixed
Parts:
- removed C2: 220n, Capacitor_SMD:C_1206_3216Metric
- removed C3: 10n, Capacitor_SMD:C_1206_3216Metric
- removed D7, D8: 1N4148WS, Diode_SMD:D_SOD-323
- removed R10: 100, Resistor_SMD:R_1206_3216Metric
- removed R13, R14: 0.22, Resistor_THT:R_Axial_Power_L38.0mm_W9.0mm_P45.72mm
- removed R15, R21: 10k, Resistor_SMD:R_1206_3216Metric
- removed U1: L6206PSO-sboxnet, sboxnet:HSOP-36-1EP_11.0x15.9mm_P0.65mm_SlugDown_ThermalVias
- added C11: 220n, Capacitor_SMD:C_1206_3216Metric, F.Cu at (134.6, 91.4)
- added C12: 10n, Capacitor_SMD:C_1206_3216Metric, F.Cu at (120.7, 90.2)
- added C13: 220n, Capacitor_SMD:C_1206_3216Metric, F.Cu at (239.6, 61.0)
- added C14: 220n, Capacitor_SMD:C_1206_3216Metric, F.Cu at (252.7, 46.5)
- added D14: 1N4148WS, Diode_SMD:D_SOD-323, F.Cu at (125.7, 88.9)
- added D15: 1N4148WS, Diode_SMD:D_SOD-323, F.Cu at (130.8, 87.6)
- added J2: cliff_FCR681465P_audiobuchse, sboxnet:CLIFF-FCR681465P, F.Cu at (29.2, 111.8)
- added JP1: SolderJumper_3_Open, Jumper:SolderJumper-3_P1.3mm_Open_RoundedPad1.0x1.5mm, F.Cu at (247.1, 43.3)
- added JP2: SolderJumper_3_Open, Jumper:SolderJumper-3_P1.3mm_Open_RoundedPad1.0x1.5mm, F.Cu at (241.2, 48.9)
- added JP3: SolderJumper_3_Open, Jumper:SolderJumper-3_P1.3mm_Open_RoundedPad1.0x1.5mm, F.Cu at (192.3, 72.2)
- added R24: 100, Resistor_SMD:R_1206_3216Metric, F.Cu at (120.7, 85.1)
- added R25: 0.22, Resistor_THT:R_Axial_Power_L38.0mm_W9.0mm_P45.72mm, F.Cu at (170.4, 18.7)
- added R26: 10k, Resistor_THT:R_Axial_Power_L38.0mm_W9.0mm_P45.72mm, F.Cu at (170.4, 39.8)
- added R27: 0.22, Resistor_THT:R_Axial_Power_L38.0mm_W9.0mm_P45.72mm, F.Cu at (220.0, 18.7)
- added R28: 10k, Resistor_THT:R_Axial_Power_L38.0mm_W9.0mm_P45.72mm, F.Cu at (170.4, 29.3)
- added U4: l6206, Package_DIP:DIP-24_W10.16mm, F.Cu at (115.6, 104.1)
- C7: value 1000u -> 2700u/25v; footprint Capacitor_THT:CP_Radial_D12.5mm_P5.00mm -> Capacitor_THT:CP_Radial_D16.0mm_P7.50mm
- C8: value 47u -> 22u/50v
- D11: value LED gn -> LED Power (gn)
- J7: footprint Connector_Audio:Jack_6.35mm_Neutrik_NRJ4HF_Horizontal -> sboxnet:CLIFF-FCR681465P
- moved SW1 243.8 mm to (270.1, 15.8)
- moved R3 228.9 mm to (259.2, 42.7), turned to 0 degrees
- moved TP9 222.3 mm to (269.9, 36.7)
- moved D5 219.5 mm to (274.6, 20.3), turned to 0 degrees
- moved C4 219.1 mm to (270.5, 24.8), turned to 0 degrees
- moved C5 218.5 mm to (259.2, 32.8)
- moved D6 218.5 mm to (274.6, 15.7), turned to 0 degrees
- moved TP5 215.6 mm to (269.9, 32.0)
- moved R23 214.9 mm to (246.8, 50.3), turned to 0 degrees
- moved C6 212.4 mm to (263.9, 25.6), turned to 0 degrees
- moved R1 211.7 mm to (241.2, 52.6), turned to 0 degrees
- moved R18 209.2 mm to (259.2, 36.1)
- moved J4 207.6 mm to (258.7, 26.3), turned to 0 degrees
- moved D4 207.0 mm to (274.5, 28.7), turned to 0 degrees
- moved TP3 202.1 mm to (264.3, 39.5)
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Connections:
- net +5V renamed Net-(J1-Pad4)
- C10 pad 1: GND -> PA2
- C10 pad 2: PA2 -> GND
- J1 pad 13: Net-(J1-Pad13) -> PB0
- J1 pad 14: Net-(J1-Pad14) -> PB1
- J1 pad 15: Net-(J1-Pad15) -> PB2
- J1 pad 21: Net-(J1-Pad21) -> /DCC_IN
- R11 pad 2: GND -> PA0
- R12 pad 1: GND -> Net-(R12-Pad1)
- R12 pad 2: Net-(R12-Pad2) -> PA2
- TP8 pad 1: VBOOT -> Net-(C11-Pad2)
- U3 pad 4: Net-(J1-Pad21) -> Net-(U3-Pad4)
Routing:
- net GND: track 297.6 -> 15.2 mm, vias 6 -> 0
- net PC3: track 212.5 -> 0.00 mm, vias 9 -> 0
- net V: track 194.6 -> 6.62 mm, vias 6 -> 0
- net +3V3: track 129.7 -> 0.00 mm, vias 3 -> 0
- net IN1: track 129.5 -> 0.00 mm, vias 7 -> 0
- net IN2: track 126.6 -> 0.00 mm, vias 8 -> 0
- net OUT2a: track 101.9 -> 0.00 mm, vias 2 -> 0
- net PA2: track 95.8 -> 0.00 mm, vias 3 -> 0
- net EN: track 85.4 -> 0.00 mm, vias 4 -> 0
- net OUT1a: track 81.4 -> 0.00 mm, vias 2 -> 0
- net VCP: track 77.7 -> 0.00 mm, vias 2 -> 0
- net PD1: track 73.7 -> 0.00 mm, vias 2 -> 0
- net VBOOT: track 72.9 -> 0.00 mm, vias 2 -> 0
- net PD0: track 72.9 -> 0.00 mm, vias 1 -> 0
- net PD2: track 68.9 -> 0.00 mm, vias 2 -> 0
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- removed copper zone on B.Cu, net GND
- removed copper zone on F.Cu, net GND
Other:
- board outline removed
- board text removed: "EN"
- board text removed: "IN1"
- board text removed: "IN2"
- board text removed: "NOTAUS"
- board text removed: "OUT1a"
- board text removed: "OUT1b"
- board text removed: "OUT2a"
- board text removed: "OUT2b"
- board text removed: "POWER"
- board text removed: "RC"
- board text removed: "RC1"
- board text removed: "Sboxnet Booster (c) 18.07.2020 Thomas Maier tom@tom.ist-im-web.de"
- board text removed: "VBOOT"
- board text removed: "Vmsg"
- board text removed: "Öffner"

Commit message: kicad 6
Other:
- net class Default removed

Commit message: entwurf fuer sboxnet-booster
Parts:
- removed C6: 220n, Capacitor_SMD:C_1206_3216Metric
- removed SW1: Öffner, Connector_PinHeader_2.54mm:PinHeader_1x03_P2.54mm_Vertical
- J7: value Power von externen 15V/4A Netzteil DS_NRJ4HF -> Conn_01x02_Male; footprint sboxnet:CLIFF-FCR681465P -> Connector_PinHeader_2.54mm:PinHeader_1x02_P2.54mm_Vertical
- R18, R19: footprint Resistor_SMD:R_1206_3216Metric -> Resistor_SMD:R_1206_3216Metric_Pad1.30x1.75mm_HandSolder
- R26, R28: footprint Resistor_THT:R_Axial_Power_L38.0mm_W9.0mm_P45.72mm -> Resistor_SMD:R_1206_3216Metric_Pad1.30x1.75mm_HandSolder
- moved R22 239.0 mm to (75.7, 178.3)
- moved D5 220.8 mm to (86.9, 136.5)
- moved R3 215.6 mm to (73.8, 152.8), turned to 180 degrees
- moved C4 214.9 mm to (73.0, 109.5)
- moved D4 208.3 mm to (93.5, 131.7)
- moved D6 206.2 mm to (97.2, 120.7)
- moved R1 201.3 mm to (73.9, 164.6), turned to 180 degrees
- moved TP3 198.5 mm to (87.9, 130.3)
- moved R23 198.4 mm to (73.8, 147.3), turned to 180 degrees
- moved R6 196.6 mm to (124.7, 182.8), turned to 180 degrees
- moved TP9 195.8 mm to (138.3, 181.6)
- moved JP1 195.6 mm to (102.5, 175.0), turned to 90 degrees
- moved C5 195.3 mm to (138.2, 186.1), turned to 90 degrees
- moved R18 194.5 mm to (135.4, 186.1), turned to -90 degrees
- moved TP2 191.1 mm to (86.5, 150.0)
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Connections:
- D4 pad 2: Net-(D4-Pad2) -> unconnected-(D4-Pad2)
- D5 pad 2: Net-(D5-Pad2) -> unconnected-(D5-Pad2)
- D6 pad 2: Net-(D6-Pad2) -> unconnected-(D6-Pad2)
- J1 pad 10: Net-(J1-Pad10) -> unconnected-(J1-Pad10)
- J1 pad 11: Net-(J1-Pad11) -> unconnected-(J1-Pad11)
- J1 pad 12: Net-(J1-Pad12) -> unconnected-(J1-Pad12)
- J1 pad 16: Net-(J1-Pad16) -> unconnected-(J1-Pad16)
- J1 pad 21: /DCC_IN -> Net-(J1-Pad21)
- J1 pad 23: Net-(J1-Pad23) -> unconnected-(J1-Pad23)
- J1 pad 24: Net-(J1-Pad24) -> unconnected-(J1-Pad24)
- J1 pad 29: Net-(J1-Pad29) -> unconnected-(J1-Pad29)
- J1 pad 30: Net-(J1-Pad30) -> unconnected-(J1-Pad30)
- J1 pad 31: Net-(J1-Pad31) -> unconnected-(J1-Pad31)
- J1 pad 32: Net-(J1-Pad32) -> unconnected-(J1-Pad32)
- J1 pad 4: Net-(J1-Pad4) -> unconnected-(J1-Pad4)
- J1 pad 8: Net-(J1-Pad8) -> unconnected-(J1-Pad8)
- J1 pad 9: Net-(J1-Pad9) -> unconnected-(J1-Pad9)
- J7 pad 1: (no net) -> GND
- J7 pad 2: (no net) -> Net-(J7-Pad2)
- R6 pad 1: Net-(R6-Pad1) -> Net-(J7-Pad2)
- R7 pad 2: Net-(R6-Pad1) -> Net-(J7-Pad2)
- TP7 pad 1: Net-(TP7-Pad1) -> Net-(D14-Pad1)
- U3 pad 1: Net-(U3-Pad1) -> unconnected-(U3-Pad1)
- U3 pad 4: Net-(U3-Pad4) -> Net-(J1-Pad21)
- U3 pad 5: Net-(U3-Pad5) -> unconnected-(U3-Pad5)
- U4 pad 1: IN2 -> IN1
- U4 pad 11: IN2 -> IN1
- U4 pad 12: IN1 -> IN2
- U4 pad 2: IN1 -> IN2
Routing:
- net GND: track 15.2 -> 629.9 mm, vias 0 -> 7
- net V: track 6.62 -> 269.0 mm, vias 0 -> 8
- net PC3: track 0.00 -> 161.5 mm, vias 0 -> 6
- net IN2: track 0.00 -> 152.0 mm, vias 0 -> 3
- net IN1: track 0.00 -> 141.9 mm, vias 0 -> 3
- net PA2: track 0.00 -> 130.1 mm, vias 0 -> 1
- net +12V: track 0.00 -> 117.4 mm, vias 0 -> 3
- net OUT2a: track 0.00 -> 115.2 mm, vias 0 -> 1
- net OUT1a: track 0.00 -> 114.5 mm, vias 0 -> 1
- net +3V3: track 0.00 -> 113.4 mm, vias 0 -> 4
- net EN: track 0.00 -> 84.8 mm, vias 0 -> 4
- net PA0: track 0.00 -> 77.4 mm, vias 0 -> 1
- net PC2: track 0.00 -> 59.2 mm, vias 0 -> 1
- net PD3: track 0.00 -> 47.2 mm, vias 0 -> 1
- net PC5: track 0.00 -> 41.0 mm, vias 0 -> 2
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- added copper zone on B.Cu, net (none)
- added copper zone on B.Cu, net GND
- added copper zone on F.Cu, net GND
Other:
- board outline added: 101.3 x 135.5 mm

Commit message: booster testpoint pc7, circuit board for out* pins to 1mm
Parts:
- removed D10: LED, LED_THT:LED_D3.0mm
- added TP12: TP, Connector_PinHeader_2.54mm:PinHeader_1x01_P2.54mm_Vertical, F.Cu at (68.7, 187.0)
- moved TP10 0.08 mm to (148.4, 97.2)
Connections:
- J1 pad 24: unconnected-(J1-Pad24) -> Net-(J1-Pad24)
Routing:
- net Net-(J1-Pad24): track 0.00 -> 20.7 mm
- net OUT2b: track 23.0 -> 27.3 mm
- net OUT2a: track 115.2 -> 112.6 mm
- net EN: track 84.8 -> 86.4 mm

Commit message: kleiner booster
Parts:
- removed C4: 220n, Capacitor_SMD:C_1206_3216Metric
- removed C8: 22u/50v, Capacitor_THT:CP_Radial_D5.0mm_P2.00mm
- removed U2: L78L12_SOT89, Package_TO_SOT_SMD:SOT-89-3
- added D10: LED, LED_THT:LED_D3.0mm, F.Cu at (104.4, 58.7)
- R1, R11, R12, R16, R17, R2, R20, R22, R23, R24, R3, R4, R5, R6, R7, R8, R9: footprint Resistor_SMD:R_1206_3216Metric -> Resistor_SMD:R_1206_3216Metric_Pad1.30x1.75mm_HandSolder
- R25, R27: footprint Resistor_THT:R_Axial_Power_L38.0mm_W9.0mm_P45.72mm -> Resistor_THT:R_Axial_DIN0614_L14.3mm_D5.7mm_P15.24mm_Horizontal
- moved R18 91.8 mm to (89.0, 106.8), turned to 180 degrees
- moved C5 89.2 mm to (89.1, 111.6), turned to 0 degrees
- moved R19 88.3 mm to (89.0, 109.2), turned to 0 degrees
- moved TP9 83.5 mm to (86.5, 116.2)
- moved R5 74.5 mm to (69.0, 143.7)
- moved C13 67.4 mm to (81.5, 102.8), turned to 0 degrees
- moved TP2 55.7 mm to (124.8, 109.5)
- moved R7 55.5 mm to (92.7, 144.8), turned to 180 degrees
- moved J7 54.6 mm to (80.4, 147.2)
- moved J5 54.4 mm to (84.6, 60.7), turned to 180 degrees
- moved R20 53.5 mm to (68.8, 89.5)
- moved TP3 52.7 mm to (124.8, 92.7)
- moved TP12 52.5 mm to (102.8, 147.0)
- moved TP1 51.7 mm to (121.0, 109.5)
- moved R27 50.3 mm to (101.6, 120.8), turned to 0 degrees
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Connections:
- J1 pad 1: +12V -> unconnected-(J1-Pad1)
Routing:
- net GND: track 629.9 -> 380.0 mm, vias 7 -> 6
- net V: track 268.8 -> 109.4 mm, vias 8 -> 6
- net +12V: track 117.1 -> 0.00 mm, vias 3 -> 0
- net PA1: track 32.7 -> 92.6 mm, vias 0 -> 3
- net PA2: track 130.1 -> 72.9 mm, vias 1 -> 0
- net PA0: track 77.4 -> 132.9 mm
- net OUT2a: track 112.6 -> 161.6 mm, vias 1 -> 0
- net IN2: track 152.0 -> 106.5 mm, vias 3 -> 2
- net PC3: track 161.5 -> 126.8 mm
- net PC5: track 41.0 -> 6.82 mm, vias 2 -> 0
- net PB2: track 11.7 -> 39.7 mm, vias 1 -> 2
- net PB1: track 13.7 -> 39.0 mm, vias 1 -> 2
- net IN1: track 141.7 -> 121.6 mm, vias 3 -> 2
- net PD3: track 47.2 -> 27.4 mm, vias 1 -> 0
- net Net-(C11-Pad2): track 31.9 -> 16.8 mm
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- removed copper zone on B.Cu, net (none)
- removed copper zone on F.Cu, net GND
Other:
- board size 101.3 x 135.5 mm -> 77.9 x 101.1 mm

Commit message: shrink booster
Parts:
- C5: value 47n -> 100n
- D4, D5, D6: value BAR42FILM -> BAT 54S
- moved R12 0.70 mm to (119.8, 125.1)
- moved C10 0.70 mm to (125.0, 125.1)
- moved R11 0.46 mm to (96.7, 109.2)
- moved TP9 0.27 mm to (86.7, 116.3)
Routing:
- net PA2: track 72.9 -> 67.9 mm
- net EN: track 71.5 -> 68.4 mm, vias 2 -> 1
- net V: track 109.4 -> 107.6 mm
- net IN2: track 106.5 -> 107.5 mm
- net Net-(R12-Pad1): track 18.5 -> 19.2 mm
- net Net-(C11-Pad2): track 16.8 -> 16.2 mm
- net PB1: track 39.0 -> 39.5 mm
- net +3V3: track 128.4 -> 127.9 mm
- added copper zone on F.Cu, net GND
Other:
- board text added: "+"
- board text added: "Cutoff"
- board text added: "Cutout"
- board text added: "IN1"
- board text added: "IN2"
- board text added: "L6206"
- board text added: "Modulcodierung"
- board text added: "NOTAUS"
- board text added: "ON"
- board text added: "OV"
- board text added: "Out1a"
- board text added: "Out2a"
- board text added: "Out2b"
- board text added: "POWER 15V/5A"
- board text added: "RC"
- board text added: "V"
- board text added: "bl"
- board text added: "ge"
- board text added: "gn"
- board text added: "rt"
- board text added: "sboxnet-booster V1 Thomas Maier tom@tom.ist-im-web.de 27.07.2022"

Commit message: sboxnet-booster-v1
Parts:
- added REF**: MountingHole_2.2mm_M2, MountingHole:MountingHole_2.2mm_M2, F.Cu at (60.7, 56.7)
- added REF**: MountingHole_2.2mm_M2, MountingHole:MountingHole_2.2mm_M2, F.Cu at (133.6, 56.6)
- added REF**: MountingHole_2.2mm_M2, MountingHole:MountingHole_2.2mm_M2, F.Cu at (60.7, 152.8)
- added REF**: MountingHole_2.2mm_M2, MountingHole:MountingHole_2.2mm_M2, F.Cu at (133.6, 152.7)
- moved J6 7.79 mm to (123.7, 60.7)
- moved D10 7.25 mm to (97.2, 58.5)
- moved D9 7.25 mm to (99.8, 63.5)
- moved R16 7.25 mm to (94.5, 61.0)
- moved R17 7.25 mm to (96.8, 67.6)
- moved R22 1.05 mm to (64.6, 151.5)
- moved TP6 0.25 mm to (132.0, 70.5)
Routing:
- net OUT2a: track 161.6 -> 152.8 mm
- net OUT1a: track 119.2 -> 113.8 mm
- net IN2: track 107.5 -> 104.7 mm, vias 2 -> 0
- net PA0: track 132.9 -> 134.8 mm
- net Net-(R22-Pad1): track 3.66 -> 2.71 mm
- net PA2: track 67.9 -> 67.1 mm
- net PB0: track 31.7 -> 31.9 mm, vias 2 -> 0
- net PB1: vias 2 -> 0
- net +3V3: vias 6 -> 7
- net PB2: vias 2 -> 0
- net IN1: vias 2 -> 0
Other:
- rule pad_to_mask_clearance: 0.051 -> 0
- board text added: "sboxnet-booster V1 Thomas Maier tom@tom.ist-im-web.de 31.07.2022"
- board text removed: "sboxnet-booster V1 Thomas Maier tom@tom.ist-im-web.de 27.07.2022"
