File: sboxnet-booster/sboxnet-booster.kicad_pcb (KiCad board)
At the start: 2 copper layers, 77.9 x 101.1 mm, 73 parts, among them J1 sboxnet-stecker_02x17, J2 cliff_FCR681465P_audiobuchse, J3 Conn_01x02_Male, J4 Conn_01x02_Male, J5 Screw_Terminal_01x04, J6 Screw_Terminal_01x04, J7 Conn_01x02_Male, U3 SN65HVD230, U4 l6206

Commit message: correct l6206 footprint, notaus as terminal block
Parts:
- D4, D5, D6: value BAT 54S -> BAT 54S NXP
- J7: value Conn_01x02_Male -> Screw_Terminal_01x02; footprint Connector_PinHeader_2.54mm:PinHeader_1x02_P2.54mm_Vertical -> TerminalBlock:TerminalBlock_Altech_AK300-2_P5.00mm
- moved J7 4.88 mm to (82.0, 142.6), turned to 180 degrees
- moved R6 0.10 mm to (92.6, 147.5)
- moved R7 0.09 mm to (92.7, 144.9)
Connections:
- J7 pad 1: GND -> Net-(J7-Pad1)
- J7 pad 2: Net-(J7-Pad2) -> GND
- R6 pad 1: Net-(J7-Pad2) -> Net-(J7-Pad1)
- R7 pad 2: Net-(J7-Pad2) -> Net-(J7-Pad1)
Routing:
- net GND: track 328.2 -> 285.2 mm, vias 6 -> 5
- net +3V3: track 127.9 -> 106.8 mm
- net PA1: track 92.3 -> 79.2 mm, vias 3 -> 0
- net Net-(J7-Pad1): track 0.00 -> 12.7 mm, vias 0 -> 1
- net Net-(J7-Pad2): track 10.8 -> 0.00 mm, vias 1 -> 0
- net PC3: track 126.6 -> 120.2 mm, vias 6 -> 4
- net PC2: track 66.8 -> 68.0 mm

Commit message: bat54s
Parts:
- D4, D5, D6: value BAT 54S NXP -> BAT 54S
Changed lines of the file:
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@@
       (effects (font (size 1 1) (thickness 0.15)))
     )
-    (fp_text value "BAT 54S NXP" (at 0 2.4) (layer "F.SilkS")
+    (fp_text value "BAT 54S" (at 0 2.4) (layer "F.SilkS")
       (effects (font (size 1 1) (thickness 0.15)))
     )
@@
       (effects (font (size 1 1) (thickness 0.15)))
     )
-    (fp_text value "BAT 54S NXP" (at -0.87 2.33) (layer "F.SilkS")
+    (fp_text value "BAT 54S" (at -0.87 2.33) (layer "F.SilkS")
       (effects (font (size 1 1) (thickness 0.15)))
     )
@@
       (effects (font (size 1 1) (thickness 0.15)))
     )
-    (fp_text value "BAT 54S NXP" (at -6.88 -0.08) (layer "F.SilkS")
-      (effects (font (size 1 1) (thickness 0.15)))
-    )
+    (fp_text value "BAT 54S" (at -6.88 -0.08) (layer "F.SilkS")
+      (effects (font (size 1 1) (thickness 0.15)))
+    )

Commit message: cleanup
Parts:
- removed C10: 1u, Capacitor_SMD:C_1206_3216Metric
- removed R25: 0.22, Resistor_THT:R_Axial_DIN0614_L14.3mm_D5.7mm_P15.24mm_Horizontal
- removed R26, R28: 10k, Resistor_SMD:R_1206_3216Metric_Pad1.30x1.75mm_HandSolder
- removed U4: l6206, Package_DIP:DIP-24_W7.62mm_Socket
- added C2: 1u, Capacitor_SMD:C_1206_3216Metric, F.Cu at (115.8, 126.5)
- added J8: Conn_01x02_Male, Connector_PinHeader_2.54mm:PinHeader_1x02_P2.54mm_Vertical, F.Cu at (128.0, 103.3)
- added J9: Conn_01x02_Male, Connector_PinHeader_2.54mm:PinHeader_1x02_P2.54mm_Vertical, F.Cu at (131.8, 103.5)
- added R10: 10k, Resistor_SMD:R_1206_3216Metric_Pad1.30x1.75mm_HandSolder, F.Cu at (79.5, 72.8)
- added R13: 10k, Resistor_SMD:R_1206_3216Metric_Pad1.30x1.75mm_HandSolder, F.Cu at (104.2, 85.5)
- added R14: 0.22, Resistor_THT:R_Axial_DIN0614_L14.3mm_D5.7mm_P15.24mm_Horizontal, F.Cu at (109.1, 86.0)
- added R15: 10k, Resistor_SMD:R_1206_3216Metric_Pad1.30x1.75mm_HandSolder, F.Cu at (115.8, 121.5)
- added TP13: TestPoint, Connector_PinHeader_2.54mm:PinHeader_1x01_P2.54mm_Vertical, F.Cu at (134.0, 110.2)
- added TP14: TestPoint, Connector_PinHeader_2.54mm:PinHeader_1x01_P2.54mm_Vertical, F.Cu at (133.8, 114.5)
- added TP15: TestPoint, Connector_PinHeader_2.54mm:PinHeader_1x01_P2.54mm_Vertical, F.Cu at (71.8, 146.5)
- added U1: L6206PSO-sboxnet, sboxnet:HSOP-36-1EP_11.0x15.9mm_P0.65mm_SlugDown_ThermalVias, F.Cu at (103.5, 99.3)
- C7: value 2700u/25v -> 2200u/25v; footprint Capacitor_THT:CP_Radial_D12.5mm_P5.00mm -> Capacitor_THT:CP_Axial_L30.0mm_D15.0mm_P35.00mm_Horizontal
- J3, J4: value Conn_01x02_Male -> Conn_01x03_Male; footprint Connector_PinHeader_2.54mm:PinHeader_1x02_P2.54mm_Vertical -> Connector_PinHeader_2.54mm:PinHeader_1x03_P2.54mm_Vertical
- R1, R2, R23, R3: value 680 -> 470
- R19: value 2.1k -> 2k
- R20: value 33k -> 10k
- moved C9 43.4 mm to (133.5, 131.5), turned to 0 degrees
- moved R11 42.2 mm to (135.0, 126.8), turned to 90 degrees
- moved C14 33.9 mm to (99.5, 115.8), turned to 0 degrees
- moved TP7 33.2 mm to (115.8, 117.0)
- moved TP10 29.7 mm to (125.0, 114.5)
- moved TP1 28.7 mm to (98.5, 127.8)
- moved TP9 25.8 mm to (61.5, 121.8)
- moved R24 25.0 mm to (106.4, 113.2), turned to 180 degrees
- moved D14 24.7 mm to (101.2, 113.1)
- moved C12 22.8 mm to (106.1, 110.7)
- moved TP3 21.3 mm to (120.2, 114.5)
- moved C13 20.8 mm to (95.8, 87.8)
- moved C5 19.9 mm to (69.8, 107.0), turned to 180 degrees
- moved D15 19.4 mm to (99.7, 84.8)
- moved J4 18.6 mm to (134.0, 92.5), turned to 0 degrees
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Connections:
- net Net-(C11-Pad2) renamed /vboot
- C12 pad 1: Net-(C12-Pad1) -> /vcp
- C9 pad 2: PA0 -> PA2
- D10 pad 2: OUT1a -> Net-(D10-Pad2)
- D9 pad 1: OUT1a -> Net-(D10-Pad2)
- J3 pad 1: OUT2b -> OUT1b
- J3 pad 2: OUT2a -> Net-(D10-Pad2)
- J4 pad 1: OUT1b -> OUT2b
- J4 pad 2: OUT1a -> Net-(J4-Pad2)
- J5 pad 1: OUT2a -> Net-(J4-Pad2)
- J5 pad 2: OUT2a -> Net-(J4-Pad2)
- J5 pad 3: OUT2a -> Net-(J4-Pad2)
- J5 pad 4: OUT2a -> Net-(J4-Pad2)
- J6 pad 1: OUT1a -> Net-(D10-Pad2)
- J6 pad 2: OUT1a -> Net-(D10-Pad2)
- J6 pad 3: OUT1a -> Net-(D10-Pad2)
- J6 pad 4: OUT1a -> Net-(D10-Pad2)
- R11 pad 1: Net-(R11-Pad1) -> PA2
- R11 pad 2: PA0 -> Net-(R11-Pad2)
- R12 pad 1: Net-(R12-Pad1) -> GND
- R12 pad 2: PA2 -> /progcl_a
- R16 pad 1: OUT2a -> Net-(J4-Pad2)
- R17 pad 1: OUT2a -> Net-(J4-Pad2)
- R17 pad 2: OUT1a -> Net-(D10-Pad2)
- R27 pad 1: GND -> /sensea
- R27 pad 2: Net-(R12-Pad1) -> GND
- TP10 pad 1: OUT2b -> OUT1a
- TP5 pad 1: OUT2a -> Net-(J4-Pad2)
- TP6 pad 1: OUT1a -> Net-(D10-Pad2)
Routing:
- net Net-(J4-Pad2): track 0.00 -> 119.3 mm
- net OUT2a: track 155.3 -> 56.3 mm, vias 0 -> 1
- net Net-(R11-Pad2): track 0.00 -> 78.8 mm, vias 0 -> 2
- net Net-(D10-Pad2): track 0.00 -> 75.9 mm
- net OUT1a: track 113.8 -> 49.6 mm, vias 1 -> 2
- net Net-(D14-Pad1): track 21.1 -> 76.1 mm, vias 0 -> 2
- net EN: track 69.9 -> 115.2 mm, vias 3 -> 4
- net PC3: track 120.2 -> 162.8 mm, vias 4 -> 6
- net IN2: track 104.7 -> 144.4 mm, vias 0 -> 2
- net OUT2b: track 33.2 -> 67.2 mm
- net /sensea: track 0.00 -> 29.8 mm, vias 0 -> 1
- net V: track 103.2 -> 131.0 mm, vias 6 -> 0
- net OUT1b: track 28.0 -> 52.3 mm, vias 0 -> 1
- net PA1: track 79.2 -> 101.2 mm, vias 0 -> 3
- net Net-(R12-Pad1): track 19.2 -> 0.00 mm
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Other:
- board text added: "A"
- board text added: "B"
- board text added: "DCC"
- board text added: "EN"
- board text added: "OUT1a"
- board text added: "OUT1b"
- board text added: "OUT2a"
- board text added: "OUT2b"
- board text added: "P"
- board text added: "VCP"
- board text removed: "+"
- board text removed: "L6206"
- board text removed: "Out1a"
- board text removed: "Out2b"
- board text removed: "bl"
- board text removed: "sboxnet-booster V2 Thomas Maier tom@tom.ist-im-web.de 20.08.2022"

Commit message: sboxnet_booster smd v3
Parts:
- D12: value SK510/310 -> SK510
- moved TP8 3.78 mm to (126.0, 80.4)
- moved J8 0.61 mm to (127.9, 103.9)
- moved J9 0.50 mm to (132.1, 103.9)
- moved J3 0.46 mm to (127.7, 92.3)
Connections:
- U1 pad 26: IN2 -> IN1
- U1 pad 27: IN1 -> IN2
Routing:
- net GND: track 268.0 -> 244.6 mm
- net /vboot: track 31.2 -> 36.9 mm
- net IN2: track 144.4 -> 148.9 mm, vias 2 -> 5
- net PA1: track 101.2 -> 104.4 mm
- net EN: track 115.2 -> 117.9 mm
- net IN1: track 130.9 -> 132.8 mm
- net OUT1b: track 52.3 -> 54.0 mm
- net Net-(D10-Pad2): track 75.9 -> 77.4 mm
- net OUT2a: track 56.3 -> 55.3 mm
- net OUT1a: track 49.6 -> 50.6 mm
- net OUT2b: track 67.2 -> 66.3 mm
- net PC3: track 162.8 -> 163.6 mm
Other:
- board text added: "+"
- board text added: "1u"
- board text added: "M(V)"
- board text added: "Out1"
- board text added: "Out2"
- board text added: "para"
- board text added: "sboxnet-booster-smd V3 Thomas Maier tom@tom.ist-im-web.de"
- board text added: "sel"
- board text added: "vboot"
- board text removed: "Out2a"
- board text removed: "V"

Commit message: sboxnet-booster-v3
Other:
- board text removed: "P"
Changed lines of the file:
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@@
     (property "Sheetname" "")
     (attr through_hole)
-    (fp_text reference "J9" (at -2.4 -0.07) (layer "F.SilkS")
+    (fp_text reference "J9" (at -1.67 -2.46) (layer "F.SilkS")
       (effects (font (size 1 1) (thickness 0.15)))
     )
@@
         (xy 8.255 -19.05)
       ) (layer "B.Cu") (width 0.1) (fill solid))
+    (fp_line (start 5.6 8.05) (end 5.6 6) (layer "F.SilkS") (width 0.12))
+    (fp_line (start 5.6 -8.05) (end 5.6 -6) (layer "F.SilkS") (width 0.12))
+    (fp_line (start -2 8.05) (end -5.6 8.05) (layer "F.SilkS") (width 0.12))
+    (fp_line (start -5.6 -6) (end -7.6 -6) (layer "F.SilkS") (width 0.12))
+    (fp_line (start -5.6 8.05) (end -5.6 6) (layer "F.SilkS") (width 0.12))
     (fp_line (start -5.6 -8.05) (end -5.6 -6) (layer "F.SilkS") (width 0.12))
-    (fp_line (start -5.6 8.05) (end -5.6 6) (layer "F.SilkS") (width 0.12))
     (fp_line (start 5.6 -8.05) (end 2 -8.05) (layer "F.SilkS") (width 0.12))
-    (fp_line (start 5.6 -8.05) (end 5.6 -6) (layer "F.SilkS") (width 0.12))
-    (fp_line (start -5.6 -6) (end -7.6 -6) (layer "F.SilkS") (width 0.12))
     (fp_line (start -2 -8.05) (end -5.6 -8.05) (layer "F.SilkS") (width 0.12))
-    (fp_line (start 5.6 8.05) (end 5.6 6) (layer "F.SilkS") (width 0.12))
-    (fp_line (start -2 8.05) (end -5.6 8.05) (layer "F.SilkS") (width 0.12))
     (fp_line (start 5.6 8.05) (end 2 8.05) (layer "F.SilkS") (width 0.12))
+    (fp_line (start 7.95 8.3) (end -7.95 8.3) (layer "F.CrtYd") (width 0.05))
+    (fp_line (start -7.95 -8.3) (end 7.95 -8.3) (layer "F.CrtYd") (width 0.05))
     (fp_line (start 7.95 8.3) (end 7.95 -8.3) (layer "F.CrtYd") (width 0.05))
-    (fp_line (start 7.95 8.3) (end -7.95 8.3) (layer "F.CrtYd") (width 0.05))
     (fp_line (start -7.95 -8.3) (end -7.95 8.3) (layer "F.CrtYd") (width 0.05))
-    (fp_line (start -7.95 -8.3) (end 7.95 -8.3) (layer "F.CrtYd") (width 0.05))
+    (fp_line (start -5.5 -6.95) (end -5.5 7.95) (layer "F.Fab") (width 0.1))
+    (fp_line (start 5.5 7.95) (end 5.5 -7.95) (layer "F.Fab") (width 0.1))
+    (fp_line (start -5.5 7.95) (end 5.5 7.95) (layer "F.Fab") (width 0.1))
+    (fp_line (start 5.5 -7.95) (end -4.5 -7.95) (layer "F.Fab") (width 0.1))
     (fp_line (start -4.5 -7.95) (end -5.5 -6.95) (layer "F.Fab") (width 0.1))
-    (fp_line (start -5.5 -6.95) (end -5.5 7.95) (layer "F.Fab") (width 0.1))
-    (fp_line (start -5.5 7.95) (end 5.5 7.95) (layer "F.Fab") (width 0.1))
-    (fp_line (start 5.5 7.95) (end 5.5 -7.95) (layer "F.Fab") (width 0.1))
-    (fp_line (start 5.5 -7.95) (end -4.5 -7.95) (layer "F.Fab") (width 0.1))
     (pad "1" smd rect (at -6.85 -5.525 90) (size 1.7 0.38) (layers "F.Cu" "F.Paste" "F.Mask")
       (net 1 "GND") (pinfunction "GND") (pintype "power_in"))
@@
     (pad "36" smd rect (at 6.85 -5.525 90) (size 1.7 0.38) (layers "F.Cu" "F.Paste" "F.Mask")
       (net 1 "GND") (pinfunction "GND") (pintype "power_in"))
+    (pad "37" smd rect (at 0 6.8425 90) (size 3.4 2.415) (layers "F.Cu" "F.Paste" "F.Mask")
+      (net 1 "GND") (pinfunction "PLANE") (pintype "power_in"))
     (pad "37" smd rect (at 0 0 90) (size 6.78 11.86) (layers "B.Cu")
+      (net 1 "GND") (pinfunction "PLANE") (pintype "power_in"))
+    (pad "37" smd rect (at 0 -6.8425 90) (size 3.4 2.415) (layers "F.Cu" "F.Paste" "F.Mask")
       (net 1 "GND") (pinfunction "PLANE") (pintype "power_in"))
     (pad "37" smd rect (at 0 0 90) (size 6.4 11.27) (layers "F.Cu" "F.Paste" "F.Mask")
       (net 1 "GND") (pinfunction "PLANE") (pintype "power_in"))
-    (pad "37" smd rect (at 0 -6.8425 90) (size 3.4 2.415) (layers "F.Cu" "F.Paste" "F.Mask")
-      (net 1 "GND") (pinfunction "PLANE") (pintype "power_in"))
-    (pad "37" smd rect (at 0 6.8425 90) (size 3.4 2.415) (layers "F.Cu" "F.Paste" "F.Mask")
-      (net 1 "GND") (pinfunction "PLANE") (pintype "power_in"))
-    (pad "38" thru_hole circle (at -0.127 -3 180) (size 4 4) (drill 3) (layers *.Cu *.Mask))
-    (pad "38" thru_hole circle (at 0.127 3 180) (size 4 4) (drill 3) (layers *.Cu *.Mask))
     (pad "38" thru_hole circle (at 0 10.16 180) (size 1.524 1.524) (drill 0.762) (layers *.Cu *.Mask))
+    (pad "38" thru_hole circle (at 0.127 0 180) (size 5 5) (drill 4) (layers *.Cu *.Mask))
     (pad "40" thru_hole circle (at 0 13.97 90) (size 1.524 1.524) (drill 0.762) (layers *.Cu *.Mask))
     (pad "42" thru_hole circle (at 0 17.78 90) (size 1.524 1.524) (drill 0.762) (layers *.Cu *.Mask))
@@
     )
   )
+  (gr_line (start 133.97 103.79) (end 133.98 101.4) (layer "F.SilkS") (width 0.12))
+  (gr_line (start 133.51 103.79) (end 133.97 103.79) (layer "F.SilkS") (width 0.12))
+  (gr_line (start 126.1 101.39) (end 126.46 101.39) (layer "F.SilkS") (width 0.12))
+  (gr_line (start 126.1 103.79) (end 126.1 101.39) (layer "F.SilkS") (width 0.12))
+  (gr_line (start 133.99 101.39) (end 133.52 101.39) (layer "F.SilkS") (width 0.12))
+  (gr_line (start 126.51 103.8) (end 126.1 103.79) (layer "F.SilkS") (width 0.12))
   (gr_rect (start 58.224 54.1655) (end 136.11 155.2745) (layer "Edge.Cuts") (width 0.05) (fill none))
   (gr_text "sboxnet-booster-smd V3\nThomas Maier\ntom@tom.ist-im-web.de\n" (at 62.4 104.33 90) (layer "F.Cu")
@@
     (effects (font (size 1 1) (thickness 0.15)))
   )
-  (gr_text "P" (at 133.75 102.5) (layer "F.SilkS")
-    (effects (font (size 1 1) (thickness 0.15)))
-  )
   (gr_text "OUT2b" (at 133.5 118.25) (layer "F.SilkS")
     (effects (font (size 1 1) (thickness 0.15)))
@@
     (effects (font (size 1 1) (thickness 0.15)))
   )
-  (gr_text "OUT2a" (at 133.75 106.25) (layer "F.SilkS")
+  (gr_text "OUT2a" (at 129.81 109.91) (layer "F.SilkS")
     (effects (font (size 1 1) (thickness 0.15)))
   )
