File: sboxnet-booster/v2-sboxnet-booster.kicad_sch (KiCad schematic)
At the start: 69 parts, among them J1 sboxnet-stecker_02x17, J2 cliff_FCR681465P_audiobuchse, J3 Conn_01x02_Male, J4 Conn_01x02_Male, J5 Screw_Terminal_01x04, J6 Screw_Terminal_01x04, J7 Conn_01x02_Male, U3 SN65HVD230, U4 l6206

Commit message: correct sboxnet-booster-v2
Parts:
- D14, D15: footprint Diode_SMD:D_SOD-123F -> Diode_SMD:D_SOD-323_HandSoldering
Changed lines of the file:
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@@
       (effects (font (size 1.27 1.27)) (justify right))
     )
-    (property "Footprint" "Diode_SMD:D_SOD-123F" (id 2) (at 181.61 97.155 0)
+    (property "Footprint" "Diode_SMD:D_SOD-323_HandSoldering" (id 2) (at 181.61 97.155 0)
       (effects (font (size 1.27 1.27)) hide)
     )
@@
       (effects (font (size 1.27 1.27)) (justify right))
     )
-    (property "Footprint" "Diode_SMD:D_SOD-123F" (id 2) (at 189.865 105.41 0)
+    (property "Footprint" "Diode_SMD:D_SOD-323_HandSoldering" (id 2) (at 189.865 105.41 0)
       (effects (font (size 1.27 1.27)) hide)
     )
@@
     )
     (path "/00000000-0000-0000-0000-000061af0c41"
-      (reference "D14") (unit 1) (value "1N4148W") (footprint "Diode_SMD:D_SOD-123F")
+      (reference "D14") (unit 1) (value "1N4148W") (footprint "Diode_SMD:D_SOD-323_HandSoldering")
     )
     (path "/00000000-0000-0000-0000-000061af30c5"
-      (reference "D15") (unit 1) (value "1N4148W") (footprint "Diode_SMD:D_SOD-123F")
+      (reference "D15") (unit 1) (value "1N4148W") (footprint "Diode_SMD:D_SOD-323_HandSoldering")
     )
     (path "/00000000-0000-0000-0000-000061b7149f"

Commit message: backup as v2
Parts:
- D14, D15: footprint Diode_SMD:D_SOD-323_HandSoldering -> Diode_SMD:D_SOD-123F
Changed lines of the file:
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@@
       (effects (font (size 1.27 1.27)) (justify right))
     )
-    (property "Footprint" "Diode_SMD:D_SOD-323_HandSoldering" (id 2) (at 181.61 97.155 0)
+    (property "Footprint" "Diode_SMD:D_SOD-123F" (id 2) (at 181.61 97.155 0)
       (effects (font (size 1.27 1.27)) hide)
     )
@@
       (effects (font (size 1.27 1.27)) (justify right))
     )
-    (property "Footprint" "Diode_SMD:D_SOD-323_HandSoldering" (id 2) (at 189.865 105.41 0)
+    (property "Footprint" "Diode_SMD:D_SOD-123F" (id 2) (at 189.865 105.41 0)
       (effects (font (size 1.27 1.27)) hide)
     )
@@
     )
     (path "/00000000-0000-0000-0000-000061af0c41"
-      (reference "D14") (unit 1) (value "1N4148W") (footprint "Diode_SMD:D_SOD-323_HandSoldering")
+      (reference "D14") (unit 1) (value "1N4148W") (footprint "Diode_SMD:D_SOD-123F")
     )
     (path "/00000000-0000-0000-0000-000061af30c5"
-      (reference "D15") (unit 1) (value "1N4148W") (footprint "Diode_SMD:D_SOD-323_HandSoldering")
+      (reference "D15") (unit 1) (value "1N4148W") (footprint "Diode_SMD:D_SOD-123F")
     )
     (path "/00000000-0000-0000-0000-000061b7149f"
