File: sboxnet-booster/v2-sboxnet-booster.kicad_sch (KiCad schematic)
At the start: 69 parts, among them J1 sboxnet-stecker_02x17, J2 cliff_FCR681465P_audiobuchse, J3 Conn_01x02_Male, J4 Conn_01x02_Male, J5 Screw_Terminal_01x04, J6 Screw_Terminal_01x04, J7 Conn_01x02_Male, U3 SN65HVD230, U4 l6206

Commit message: v2-sboxnet-booster
Parts:
- removed J7: Conn_01x02_Male, Connector_PinHeader_2.54mm:PinHeader_1x02_P2.54mm_Vertical, symbol Connector:Conn_01x02_Male
- added J7: Screw_Terminal_01x02, TerminalBlock:TerminalBlock_Altech_AK300-2_P5.00mm, symbol Connector:Screw_Terminal_01x02
- D4, D5, D6: value BAT 54S NXP -> BAT 54S
Connections:
- net GND: now also J7.2 (Pin_2)
- net at R6.1, R7.2: now also J7.1 (Pin_1)
Changed lines of the file:
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@@
     (in_bom yes) (on_board yes)
     (property "Reference" "D5" (id 0) (at 86.7664 80.2386 0))
-    (property "Value" "BAT 54S NXP" (id 1) (at 86.7664 82.55 0))
+    (property "Value" "BAT 54S" (id 1) (at 86.7664 82.55 0))
     (property "Footprint" "Package_TO_SOT_SMD:SOT-23_Handsoldering" (id 2) (at 86.7664 91.821 0)
       (effects (font (size 1.27 1.27)) hide)
@@
       (effects (font (size 1.27 1.27)) (justify right))
     )
-    (property "Value" "BAT 54S NXP" (id 1) (at 93.9292 104.5718 90)
+    (property "Value" "BAT 54S" (id 1) (at 93.9292 104.5718 90)
       (effects (font (size 1.27 1.27)) (justify right))
     )
@@
     (in_bom yes) (on_board yes)
     (property "Reference" "D4" (id 0) (at 73.8632 91.567 0))
-    (property "Value" "BAT 54S NXP" (id 1) (at 73.8632 93.8784 0))
+    (property "Value" "BAT 54S" (id 1) (at 73.8632 93.8784 0))
     (property "Footprint" "Package_TO_SOT_SMD:SOT-23_Handsoldering" (id 2) (at 73.8632 92.6338 0)
       (effects (font (size 1.27 1.27)) hide)
@@
     (pin "1")
   )
-  (symbol (lib_id "Connector:Conn_01x02_Male") (at 84.328 128.016 180) (unit 1)
-    (in_bom yes) (on_board yes)
-    (property "Reference" "J7" (id 0) (at 85.725 131.699 0)
-      (effects (font (size 1.27 1.27)) (justify right))
-    )
-    (property "Value" "Conn_01x02_Male" (id 1) (at 84.582 133.731 0)
-      (effects (font (size 1.27 1.27)) (justify right))
-    )
-    (property "Footprint" "Connector_PinHeader_2.54mm:PinHeader_1x02_P2.54mm_Vertical" (id 2) (at 84.328 128.016 0)
-      (effects (font (size 1.27 1.27)) hide)
-    )
-    (property "Datasheet" "~" (id 3) (at 84.328 128.016 0)
+  (symbol (lib_id "Connector:Screw_Terminal_01x02") (at 84.328 125.476 0) (unit 1)
+    (in_bom yes) (on_board yes) (fields_autoplaced)
+    (property "Reference" "J7" (id 0) (at 86.36 125.9113 0)
+      (effects (font (size 1.27 1.27)) (justify left))
+    )
+    (property "Value" "Screw_Terminal_01x02" (id 1) (at 86.36 128.4482 0)
+      (effects (font (size 1.27 1.27)) (justify left))
+    )
+    (property "Footprint" "TerminalBlock:TerminalBlock_Altech_AK300-2_P5.00mm" (id 2) (at 84.328 125.476 0)
+      (effects (font (size 1.27 1.27)) hide)
+    )
+    (property "Datasheet" "~" (id 3) (at 84.328 125.476 0)
       (effects (font (size 1.27 1.27)) hide)
     )
@@
     )
     (path "/00000000-0000-0000-0000-00005f1b960f"
-      (reference "D4") (unit 1) (value "BAT 54S NXP") (footprint "Package_TO_SOT_SMD:SOT-23_Handsoldering")
+      (reference "D4") (unit 1) (value "BAT 54S") (footprint "Package_TO_SOT_SMD:SOT-23_Handsoldering")
     )
     (path "/00000000-0000-0000-0000-00005f0e2174"
-      (reference "D5") (unit 1) (value "BAT 54S NXP") (footprint "Package_TO_SOT_SMD:SOT-23_Handsoldering")
+      (reference "D5") (unit 1) (value "BAT 54S") (footprint "Package_TO_SOT_SMD:SOT-23_Handsoldering")
     )
     (path "/00000000-0000-0000-0000-00005f139ee6"
-      (reference "D6") (unit 1) (value "BAT 54S NXP") (footprint "Package_TO_SOT_SMD:SOT-23_Handsoldering")
+      (reference "D6") (unit 1) (value "BAT 54S") (footprint "Package_TO_SOT_SMD:SOT-23_Handsoldering")
     )
     (path "/00000000-0000-0000-0000-00005dba95ff"
@@
       (reference "J6") (unit 1) (value "Screw_Terminal_01x04") (footprint "TerminalBlock:TerminalBlock_Altech_AK300-4_P5.00mm")
     )
-    (path "/df854d90-91a6-497c-aba1-6c00d8cc77a4"
-      (reference "J7") (unit 1) (value "Conn_01x02_Male") (footprint "Connector_PinHeader_2.54mm:PinHeader_1x02_P2.54mm_Vertical")
+    (path "/ec759541-1088-4e24-9c36-8a916e48ae55"
+      (reference "J7") (unit 1) (value "Screw_Terminal_01x02") (footprint "TerminalBlock:TerminalBlock_Altech_AK300-2_P5.00mm")
     )
     (path "/00000000-0000-0000-0000-000061b2babb"
