File: sboxnet-booster/v2-sboxnet-booster.kicad_pcb (KiCad board)
At the start: 2 copper layers, 77.9 x 101.1 mm, 73 parts, among them J1 sboxnet-stecker_02x17, J2 cliff_FCR681465P_audiobuchse, J3 Conn_01x02_Male, J4 Conn_01x02_Male, J5 Screw_Terminal_01x04, J6 Screw_Terminal_01x04, J7 Conn_01x02_Male, U3 SN65HVD230, U4 l6206

Commit message: correct sboxnet-booster-v2
Parts:
- D14, D15: footprint Diode_SMD:D_SOD-123F -> Diode_SMD:D_SOD-323
- moved TP3 2.46 mm to (120.8, 95.2)
- moved D15 1.09 mm to (116.8, 91.8)
- moved D14 0.45 mm to (112.9, 91.8)
- moved J3 0.34 mm to (130.2, 86.3)
- moved C11 0.13 mm to (113.3, 94.0)
Routing:
- net EN: track 69.9 -> 67.3 mm
Other:
- board text added: "sboxnet-booster V2 Thomas Maier tom@tom.ist-im-web.de 16.08.2022"
- board text removed: "sboxnet-booster V2 Thomas Maier tom@tom.ist-im-web.de 20.08.2022"

Commit message: backup as v2
Parts:
- D14, D15: footprint Diode_SMD:D_SOD-323 -> Diode_SMD:D_SOD-123F
- moved TP3 2.46 mm to (122.2, 93.2)
- moved D15 1.09 mm to (117.9, 91.5)
- moved D14 0.45 mm to (113.3, 91.5)
- moved J3 0.34 mm to (130.5, 86.2)
- moved C11 0.13 mm to (113.3, 93.8)
Routing:
- net EN: track 67.3 -> 69.9 mm
Other:
- board text added: "sboxnet-booster V2 Thomas Maier tom@tom.ist-im-web.de 20.08.2022"
- board text removed: "sboxnet-booster V2 Thomas Maier tom@tom.ist-im-web.de 16.08.2022"

Commit message: v2-sboxnet-booster
Parts:
- J7: value Conn_01x02_Male -> Screw_Terminal_01x02; footprint Connector_PinHeader_2.54mm:PinHeader_1x02_P2.54mm_Vertical -> TerminalBlock:TerminalBlock_Altech_AK300-2_P5.00mm
- moved J7 4.88 mm to (82.0, 142.6), turned to 180 degrees
- moved R6 0.10 mm to (92.6, 147.5)
- moved R7 0.09 mm to (92.7, 144.9)
Connections:
- J7 pad 1: GND -> Net-(J7-Pad1)
- J7 pad 2: Net-(J7-Pad2) -> GND
- R6 pad 1: Net-(J7-Pad2) -> Net-(J7-Pad1)
- R7 pad 2: Net-(J7-Pad2) -> Net-(J7-Pad1)
Routing:
- net GND: track 328.2 -> 285.2 mm, vias 6 -> 5
- net +3V3: track 127.9 -> 106.8 mm
- net PA1: track 92.3 -> 79.2 mm, vias 3 -> 0
- net Net-(J7-Pad1): track 0.00 -> 12.7 mm, vias 0 -> 1
- net Net-(J7-Pad2): track 10.8 -> 0.00 mm, vias 1 -> 0
- net PC3: track 126.6 -> 120.2 mm, vias 6 -> 4
- net PC2: track 66.8 -> 68.0 mm
