File: sboxnet2usb/sboxnet2usb.kicad_pcb (KiCad board)
At the start: 2 copper layers, 107.2 x 47.8 mm, 54 parts, among them J1 USB_A, J2 cliff_FCR681465P_audiobuchse, J3 8P8C, J4 8P8C, J5 Conn_01x02_Male, J6 Conn_01x02_Male, J7 Screw_Terminal_01x02, J8 Screw_Terminal_01x02, U1 ATmega32U2-AU, U2 wannenstecker6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

Commit message: kicad 5 -> 6
Other:
- net class Default removed
