File: sboxnet-gbm2/sboxnet-gbm2.kicad_sch (KiCad schematic)
At the start: 23 parts, among them J1 sboxnet-stecker_02x17, J2 Conn_02x03_Odd_Even, U1 QS4A_0303S1.5UP, U2 ATxmega32A4U-A, Y1 Crystal

Commit message: gbm2-schema
Parts:
- removed C1: C_Polarized, symbol Device:C_Polarized
- removed C2: 1u, symbol Device:C_Polarized
- removed C3, C4: 22p, symbol Device:C
- removed C5, C6, C7: 100n, symbol Device:C
- removed J2: Conn_02x03_Odd_Even, symbol Connector_Generic:Conn_02x03_Odd_Even
- removed J?: sboxnet-buchse_02x17, sboxnet:connector_2x17, symbol sboxnet:sboxnet-buchse_02x17
- removed JP1, JP2, JP3, JP4: SolderJumper_3_Open, symbol Jumper:SolderJumper_3_Open
- removed L1: Ferrit, symbol Device:L
- removed U1: QS4A_0303S1.5UP, symbol sboxnet:QS4A_0303S1.5UP
- removed U2: ATxmega32A4U-A, Package_QFP:TQFP-44_10x10mm_P0.8mm, symbol MCU_Microchip_ATmega:ATxmega32A4U-A
- removed Y1: Crystal, symbol Device:Crystal
- added D10, D11, D16, D17, D21, D22, D23, D24, D3, D4, D5, D6, D7, D8: SB340, Diode_SMD:D_SMC_Handsoldering, symbol Device:D_Schottky
- added D12, D13, D14, D15, D18, D19, D20, D9: LED, symbol Device:LED
- added JP1, JP2, JP3, JP4: Jumper_2_Open, symbol Jumper:Jumper_2_Open
- added R10, R16, R21, R23, R5, R7: 22/1W, symbol Device:R
- added R11, R13, R14, R15, R17, R19, R20, R9: R, symbol Device:R
- added R12, R18, R22, R24, R4, R6, R8: 1k, symbol Device:R
- R3: value 680 -> 22/1W
Connections:
- net +3.3V: now also R11.1, R13.1, R14.1, R15.1, R17.1, R19.1, R20.1, R9.1
- net GND: now also J1.2 (Pin_2), JP1.1 (A), JP2.1 (A), JP3.1 (A), JP4.1 (A)
- net PB0: now also JP1.2 (B)
- net PB1: now also JP2.2 (B)
- net PB2: now also JP3.2 (B)
- net PB3: now also JP4.2 (B)
- net sens_0: now also J1.5 (Pin_5)
- net sens_5: now reaches J1.10 (Pin_10)
- net sens_5: now also R18.2
- net sens_6: now reaches J1.11 (Pin_11)
- net sens_6: now also R22.2
- net sens_7: now reaches J1.12 (Pin_12)
- net sens_7: now also R24.2
- net l0: now reaches J1.25 (Pin_25)
- net l0: now also D9.1 (K)
- net l1: now reaches J1.26 (Pin_26)
- net l1: now also D12.1 (K)
- net l2: now reaches J1.27 (Pin_27)
- net l2: now also D13.1 (K)
- net l3: now reaches J1.28 (Pin_28)
- net l3: now also D14.1 (K)
- net l4: now reaches J1.29 (Pin_29)
- net l4: now also D15.1 (K), D18.1 (K), D19.1 (K), D20.1 (K)
- net l5: now reaches J1.30 (Pin_30)
- net l6: now reaches J1.31 (Pin_31)
- net l7: now reaches J1.32 (PD7)
- net sens_1: now reaches J1.6 (Pin_6)
- net sens_1: now also R4.2
- net sens_2: now reaches J1.7 (Pin_7)
- net sens_2: now also R6.2
- net sens_3: now reaches J1.8 (Pin_8)
- net sens_3: now also R8.2
- net sens_4: now reaches J1.9 (Pin_9)
- net sens_4: now also R12.2
- net +3.3VP: no longer names the net of R3.1
- net +3.3VP: now also D3.2 (A)
- net GND1: no longer names the net of D2.2 (A), R1.1
- net GND1: no longer D1.1 (K), R3.2
- net dcc1: no longer names the net of D2.1 (K), R1.2
- net dcc1: no longer D1.2 (A)
- new net: D16.2 (A), R16.1
- new net: D16.1 (K), R16.2
- new net: D7.1 (K), R7.2
- new net: D7.2 (A), R7.1
- new net: D3.1 (K), R3.2
- new net: D10.1 (K), R10.2
- new net: D10.2 (A), R10.1
- new net: D5.1 (K), R5.2
- new net: D5.2 (A), R5.1
- new net: D13.2 (A), R13.2
- new net: D18.2 (A), R17.2
- new net: D19.2 (A), R19.2
- new net: D12.2 (A), R11.2
- new net: D20.2 (A), R20.2
- new net: D15.2 (A), R15.2
- new net: D9.2 (A), R9.2
- new net: D14.2 (A), R14.2
- new net: D23.2 (A), R23.1
- new net: D23.1 (K), R23.2
- new net: D21.1 (K), R21.2
- new net: D21.2 (A), R21.1
- no-connect marks 4 -> 2
Other:
- note removed: "DC/DC 3.3V/3.3V Isolated, Unregulated"
- moved on the sheet: D2, R1, R2
