File: sboxnet/sboxnet.kicad_sch (KiCad schematic)
At the start: 8 parts

Commit message: sboxnet schema
Parts:
- added T? (x2): Transformer_1P_1S, symbol Device:Transformer_1P_1S
- added U? (x2): 6N137, Package_DIP:DIP-8_W7.62mm, symbol Isolator:6N137
Connections:
- net +15v: now also T?.4 (SB), U?.8 (VCC)
- net GND: now also T?.3 (SA), U?.3 (C), U?.5 (GND)
Other:
- note added: "dcc_1"
- note added: "dcc_GND"
- note added: "sboxnet2usb"
- note added: "sboxnet_GND"
