File: sboxnet-modul/sboxnet-modul.kicad_sch (KiCad schematic)
At the start: 35 parts

Commit message: sboxnet-modul v5
Parts:
- removed J3: (no value), symbol Connector:Conn_01x04_Female
- C1, C10, C4, C5, C6: value (none) -> 100n; footprint (none) -> Capacitor_SMD:C_1206_3216Metric_Pad1.42x1.75mm_HandSolder
- C2: value (none) -> 10u; footprint (none) -> Capacitor_SMD:C_1206_3216Metric_Pad1.42x1.75mm_HandSolder
- C3: value (none) -> 10u; footprint (none) -> Capacitor_SMD:C_1206_3216Metric
- C7: value (none) -> 1u; footprint (none) -> Capacitor_SMD:C_1206_3216Metric_Pad1.42x1.75mm_HandSolder
- C8, C9: value (none) -> 15p; footprint (none) -> Capacitor_SMD:C_1206_3216Metric_Pad1.42x1.75mm_HandSolder
- D1: value (none) -> SKL13B; footprint (none) -> Diode_SMD:D_SMB_Handsoldering
- D2, D3, D4, D5: value (none) -> LED; footprint (none) -> LED_SMD:LED_1206_3216Metric_Pad1.42x1.75mm_HandSolder
- J1: value (none) -> Conn_01x03; footprint (none) -> Connector_PinHeader_2.54mm:PinHeader_1x03_P2.54mm_Vertical
- J2: value (none) -> Conn_02x03_Odd_Even; footprint (none) -> sboxnet:wannenstecker_gerade_6pin
- J4, J5: value (none) -> 8P8C; footprint (none) -> sboxnet:8p8c-mebp
- J6: value (none) -> sboxnet-buchse_2x17; footprint (none) -> sboxnet:sboxnet-buchse-2x17
- L1: value (none) -> Ferrit 60Ohm; footprint (none) -> Inductor_SMD:L_1206_3216Metric_Pad1.42x1.75mm_HandSolder
- R1, R3, R4, R7: value (none) -> 470; footprint (none) -> Resistor_SMD:R_1206_3216Metric_Pad1.42x1.75mm_HandSolder
- R2: value (none) -> 0; footprint (none) -> Resistor_SMD:R_1206_3216Metric_Pad1.42x1.75mm_HandSolder
- R5: value (none) -> 1k; footprint (none) -> Resistor_SMD:R_1206_3216Metric_Pad1.42x1.75mm_HandSolder
- R6: value (none) -> 10k; footprint (none) -> Resistor_SMD:R_1206_3216Metric_Pad1.42x1.75mm_HandSolder
- SW1: value (none) -> SW_Push; footprint (none) -> sboxnet:JTP-1130
- U1: value (none) -> MCP1703A-3302_SOT223; footprint (none) -> Package_TO_SOT_SMD:SOT-223-3_TabPin2
- U2: value (none) -> MCP1703A-5002_SOT223; footprint (none) -> Package_TO_SOT_SMD:SOT-223-3_TabPin2
- U3: value (none) -> SN65HVD230; footprint (none) -> Package_SO:SOIC-8_3.9x4.9mm_P1.27mm
- U4: value (none) -> ATxmega128A4U-AU; footprint (none) -> Package_QFP:TQFP-44_10x10mm_P0.8mm
- Y1: value (none) -> 16MHz; footprint (none) -> Crystal:Crystal_HC49-U_Vertical

Commit message: fix
Parts:
- C1, C10, C2, C4, C5, C6, C7, C8, C9: footprint Capacitor_SMD:C_1206_3216Metric_Pad1.42x1.75mm_HandSolder -> Capacitor_SMD:C_1206_3216Metric_Pad1.33x1.80mm_HandSolder
- R1, R2, R3, R4, R5, R6, R7: footprint Resistor_SMD:R_1206_3216Metric_Pad1.42x1.75mm_HandSolder -> Resistor_SMD:R_1206_3216Metric_Pad1.30x1.75mm_HandSolder

Commit message: sboxnet modul v6.2
Parts:
- removed J1: Conn_01x03, Connector_PinHeader_2.54mm:PinHeader_1x03_P2.54mm_Vertical, symbol Connector_Generic:Conn_01x03
Connections:
- net +7V: now also D1.2 (A)
- net at C1.2, U2.1 (VI): no longer D1.1 (K)
Other:
- moved on the sheet: D1
Changed lines of the file:
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@@
   (junction (at 59.563 64.643) (diameter 0) (color 0 0 0 0)
   )
-  (junction (at 33.401 33.655) (diameter 0) (color 0 0 0 0)
-  )
   (junction (at 74.041 64.77) (diameter 0) (color 0 0 0 0)
   )
@@
   )
   (junction (at 98.425 64.897) (diameter 0) (color 0 0 0 0)
+  )
+  (junction (at 33.3756 33.6296) (diameter 0) (color 0 0 0 0)
   )
   (junction (at 43.561 64.516) (diameter 0) (color 0 0 0 0)
@@
     (stroke (width 0) (type default) (color 0 0 0 0))
   )
+  (wire (pts (xy 33.3756 31.75) (xy 33.3756 33.6296))
+    (stroke (width 0) (type default) (color 0 0 0 0))
+  )
   (wire (pts (xy 191.135 57.658) (xy 196.088 57.658))
     (stroke (width 0) (type default) (color 0 0 0 0))
@@
     (stroke (width 0) (type default) (color 0 0 0 0))
   )
-  (wire (pts (xy 31.369 26.035) (xy 35.941 26.035))
+  (wire (pts (xy 30.48 31.75) (xy 33.3756 31.75))
     (stroke (width 0) (type default) (color 0 0 0 0))
   )
@@
   )
   (wire (pts (xy 51.816 64.516) (xy 59.563 64.516))
-    (stroke (width 0) (type default) (color 0 0 0 0))
-  )
-  (wire (pts (xy 28.829 33.655) (xy 33.401 33.655))
     (stroke (width 0) (type default) (color 0 0 0 0))
   )
@@
     )
   )
-  (global_label "+V" (shape input) (at 35.941 26.035 0) (fields_autoplaced)
-    (effects (font (size 1.27 1.27)) (justify left))
-    (property "Referenzen zwischen Schaltplänen" "${INTERSHEET_REFS}" (id 0) (at 0 0 0)
-      (effects (font (size 1.27 1.27)) hide)
-    )
-  )
   (global_label "PD3" (shape input) (at 191.135 57.658 180) (fields_autoplaced)
     (effects (font (size 0.9906 0.9906)) (justify right))
@@
     )
   )
-  (global_label "+7V" (shape input) (at 26.289 26.035 270) (fields_autoplaced)
-    (effects (font (size 0.9906 0.9906)) (justify right))
-    (property "Referenzen zwischen Schaltplänen" "${INTERSHEET_REFS}" (id 0) (at 0 0 0)
+  (global_label "+7V" (shape input) (at 30.48 24.13 90) (fields_autoplaced)
+    (effects (font (size 0.9906 0.9906)) (justify left))
+    (property "Referenzen zwischen Schaltplänen" "${INTERSHEET_REFS}" (id 0) (at 56.769 50.165 0)
       (effects (font (size 1.27 1.27)) hide)
     )
@@
     (pin "1")
   )
-  (symbol (lib_id "Device:D_Schottky") (at 28.829 29.845 90) (unit 1)
-    (in_bom yes) (on_board yes)
-    (property "Reference" "D1" (id 0) (at 30.8356 28.6766 90)
-      (effects (font (size 1.27 1.27)) (justify right))
-    )
-    (property "Value" "SKL13B" (id 1) (at 30.8356 30.988 90)
-      (effects (font (size 1.27 1.27)) (justify right))
-    )
-    (property "Footprint" "Diode_SMD:D_SMB_Handsoldering" (id 2) (at 28.829 29.845 0)
-      (effects (font (size 1.27 1.27)) hide)
-    )
-    (property "Datasheet" "~" (id 3) (at 28.829 29.845 0)
+  (symbol (lib_id "Device:D_Schottky") (at 30.48 27.94 90) (unit 1)
+    (in_bom yes) (on_board yes)
+    (property "Reference" "D1" (id 0) (at 32.4866 26.7716 90)
+      (effects (font (size 1.27 1.27)) (justify right))
+    )
+    (property "Value" "SKL13B" (id 1) (at 32.4866 29.083 90)
+      (effects (font (size 1.27 1.27)) (justify right))
+    )
+    (property "Footprint" "Diode_SMD:D_SMB_Handsoldering" (id 2) (at 30.48 27.94 0)
+      (effects (font (size 1.27 1.27)) hide)
+    )
+    (property "Datasheet" "~" (id 3) (at 30.48 27.94 0)
       (effects (font (size 1.27 1.27)) hide)
     )
@@
     (in_bom yes) (on_board yes)
     (property "Reference" "U2" (id 0) (at 44.323 26.289 0))
-    (property "Value" "MCP1703A-5002_SOT223" (id 1) (at 46.482 28.067 0))
+    (property "Value" "MCP1703A-5002_SOT223" (id 1) (at 44.8564 24.5364 0))
     (property "Footprint" "Package_TO_SOT_SMD:SOT-223-3_TabPin2" (id 2) (at 44.196 28.575 0)
       (effects (font (size 1.27 1.27)) hide)
@@
       (effects (font (size 1.27 1.27)) hide)
     )
-    (property "Value" "PWR_FLAG" (id 1) (at 35.179 29.2608 0))
+    (property "Value" "PWR_FLAG" (id 1) (at 40.4368 30.6832 0))
     (property "Footprint" "" (id 2) (at 35.179 33.655 0)
       (effects (font (size 1.27 1.27)) hide)
@@
     (pin "8")
     (pin "9")
-  )
-  (symbol (lib_id "Connector_Generic:Conn_01x03") (at 28.829 20.955 90) (unit 1)
-    (in_bom yes) (on_board yes)
-    (property "Reference" "J1" (id 0) (at 33.6042 21.8694 90)
-      (effects (font (size 1.27 1.27)) (justify right))
-    )
-    (property "Value" "Conn_01x03" (id 1) (at 33.6042 24.1808 90)
-      (effects (font (size 1.27 1.27)) (justify right))
-    )
-    (property "Footprint" "Connector_PinHeader_2.54mm:PinHeader_1x03_P2.54mm_Vertical" (id 2) (at 28.829 20.955 0)
-      (effects (font (size 1.27 1.27)) hide)
-    )
-    (property "Datasheet" "~" (id 3) (at 28.829 20.955 0)
-      (effects (font (size 1.27 1.27)) hide)
-    )
-    (pin "1")
-    (pin "2")
-    (pin "3")
   )
   (symbol (lib_id "Interface_CAN_LIN:SN65HVD230") (at 50.419 132.461 180) (unit 1)
@@
       (reference "D5") (unit 1) (value "LED") (footprint "LED_SMD:LED_1206_3216Metric_Pad1.42x1.75mm_HandSolder")
     )
-    (path "/00000000-0000-0000-0000-00005d99fa51"
-      (reference "J1") (unit 1) (value "Conn_01x03") (footprint "Connector_PinHeader_2.54mm:PinHeader_1x03_P2.54mm_Vertical")
-    )
     (path "/00000000-0000-0000-0000-0000605a2020"

Commit message: sboxnet modul V6
Parts:
- C3: footprint Capacitor_SMD:C_1206_3216Metric -> Capacitor_SMD:C_1206_3216Metric_Pad1.33x1.80mm_HandSolder
Connections:
- net at D1.1 (K): now also C1.2, U2.1 (VI)
Other:
- moved on the sheet: C1, D1

Commit message: sboxnet Modul v6 with some mods
Connections:
- net +V: no longer names the net of J6.1 (Pin_1)
- no-connect marks 1 -> 4
Changed lines of the file:
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@@
   (junction (at 66.929 64.643) (diameter 0) (color 0 0 0 0)
   )
+  (no_connect (at 73.66 91.694))
   (no_connect (at 60.579 129.921))
+  (no_connect (at 208.788 90.678))
+  (no_connect (at 60.96 91.694))
   (wire (pts (xy 34.798 34.29) (xy 36.83 34.29))
     (stroke (width 0) (type default) (color 0 0 0 0))
@@
     (effects (font (size 0.9906 0.9906)) (justify left))
     (property "Referenzen zwischen Schaltplänen" "${INTERSHEET_REFS}" (id 0) (at 0 0 0)
-      (effects (font (size 1.27 1.27)) hide)
-    )
-  )
-  (global_label "+V" (shape input) (at 208.788 90.678 0) (fields_autoplaced)
-    (effects (font (size 0.9906 0.9906)) (justify left))
-    (property "Referenzen zwischen Schaltplänen" "${INTERSHEET_REFS}" (id 0) (at 0 0 0)
