File: sboxnet-modul/sboxnet-modul.kicad_pcb (KiCad board)
At the start: 2 copper layers, 49.6 x 46.2 mm, 33 parts, among them J2 Conn_02x03_Odd_Even, J4 8P8C, J5 8P8C, J6 sboxnet-buchse_2x17, SW1 SW_Push, U1  3.3V MCP1703A-3302_SOT223, U2  5V MCP1703A-5002_SOT223, U3 SN65HVD230, U4 ATxmega128A4U-AU, Y1 16MHz

Commit message: sboxnet Modul v6 with some mods
Other:
- board text added: "PDI"
- board text added: "action"
- board text added: "active"
- board text added: "error"
Changed lines of the file:
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@@
       (effects (font (size 1 1) (thickness 0.15)))
     )
-    (fp_text value "ATxmega128A4U-AU" (at 0 7.45 135) (layer "F.Fab")
+    (fp_text value "ATxmega128A4U-AU" (at -7.36381 0.35921 225) (layer "F.SilkS")
       (effects (font (size 1 1) (thickness 0.15)))
     )
@@
       (effects (font (size 1 1) (thickness 0.15)))
     )
-    (fp_text value "SN65HVD230" (at 0 3.4 90) (layer "F.Fab")
+    (fp_text value "SN65HVD230" (at 0 3.4 90) (layer "F.SilkS")
       (effects (font (size 1 1) (thickness 0.15)))
     )
@@
   )
   (gr_circle (center 92.5576 90.8558) (end 92.791776 90.8558) (layer "F.SilkS") (width 0.15) (fill none))
+  (gr_circle (center 112.776 112.776) (end 113.010176 112.776) (layer "F.SilkS") (width 0.15) (fill none))
   (gr_line (start 125.73 121.92) (end 76.2 121.92) (layer "Edge.Cuts") (width 0.1))
   (gr_line (start 76.2 121.92) (end 76.1746 75.7682) (layer "Edge.Cuts") (width 0.1))
@@
     (effects (font (size 1 1) (thickness 0.1)))
   )
-  (gr_text "gn" (at 83.8454 113.8428) (layer "F.SilkS")
+  (gr_text "gn" (at 83.82 113.538 90) (layer "F.SilkS")
+    (effects (font (size 1 1) (thickness 0.15)))
+  )
+  (gr_text "PDI" (at 96.012 113.157) (layer "F.SilkS")
+    (effects (font (size 1 1) (thickness 0.1)))
+  )
+  (gr_text "error" (at 86.487 110.617 90) (layer "F.SilkS")
+    (effects (font (size 1 1) (thickness 0.15)))
+  )
+  (gr_text "active" (at 83.82 110.109 90) (layer "F.SilkS")
     (effects (font (size 1 1) (thickness 0.15)))
   )
@@
     (effects (font (size 1 1) (thickness 0.15)))
   )
-  (gr_text "rt" (at 86.5632 113.9952) (layer "F.SilkS")
+  (gr_text "action" (at 92.202 114.046) (layer "F.SilkS")
     (effects (font (size 1 1) (thickness 0.15)))
   )
+  (gr_text "rt" (at 86.487 114.046 90) (layer "F.SilkS")
+    (effects (font (size 1 1) (thickness 0.15)))
+  )

Commit message: sboxnet Modul v6 fertig
Other:
- board text added: "bl 3.3V"
- board text added: "or 5V"
- board text removed: "bl"
- board text removed: "or"
